File: 03 - PCB/DAB_PCB/test/DAB_Template4Students.kicad_sch (KiCad schematic)
At the start: 106 parts, among them IC1 UCC27288DR, IC2 UCC27288DR, IC3 UCC27288DR, IC4 UCC27288DR

Commit message: power supply and measuremtents schematics
Parts:
- added C10, C11, C12, C13, C14, C15, C16, C17, C18, C19, C20, C25, C5, C6, C7, C8, C9, C_fil1, C_fil2, C_fil3, C_vdd5, C_vdd6, C_vdd8, C_vdd9, Csens1, Csens2: Put Value Here!, C__Users_Jiasheng_OneDrive - epfl.ch_Jiasheng_EPFL_03_SideWork_08_TA_AlitumTemplate_DAB_Template_DAB_PCB.PcbLib:SM/1206, symbol DAB_EE365:root_1_Capacitor (SMD)_DAB_EE365.SchLib
- added D2, D3, D4, D5: ES2C, C__Users_Jiasheng_OneDrive - epfl.ch_Jiasheng_EPFL_03_SideWork_08_TA_Altium_Template_for_EE365_student_PCB1.PcbLib:DIOM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, symbol DAB_EE365:root_0_Schottky Diode_DAB_EE365.SchLib
- added IC10, IC9: MCP6241-E_P, C__Users_Jiasheng_OneDrive - epfl.ch_Documents_AltiumLL_SamacSys.PcbLib:DIP781W56P254L950H533Q8N, symbol DAB_EE365:root_0_MCP6241-E_P_DAB_EE365.SchLib
- added IC11: AZ1117IH-3.3TRG1, C__Users_Jiasheng_OneDrive - epfl.ch_Documents_AltiumLL_SamacSys.PcbLib:SOT230P700X180-4N, symbol DAB_EE365:root_0_AZ1117IH-3.3TRG1_DAB_EE365.SchLib
- added IC12: UA78L12ACDR, C__Users_Jiasheng_OneDrive - epfl.ch_Jiasheng_EPFL_03_SideWork_08_TA_Altium_Template_for_EE365_student_PCB1.PcbLib:SOIC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, symbol DAB_EE365:root_0_UA78L12ACDR_DAB_EE365.SchLib
- added IC5, IC6, IC7, IC8: INA201AID, C__Users_Jiasheng_OneDrive - epfl.ch_Documents_AltiumLL_SamacSys.PcbLib:SOIC127P600X175-8N, symbol DAB_EE365:root_0_INA201AID_DAB_EE365.SchLib
- added LED1, LED2, LED3, LED4, LED5: WP710A10LGD, C__Users_Jiasheng_OneDrive - epfl.ch_Documents_AltiumLL_SamacSys.PcbLib:WP710A10LGD, symbol DAB_EE365:root_2_WP710A10LGD_DAB_EE365.SchLib
- added PS1, PS3: 173951275, C__Users_Jiasheng_OneDrive - epfl.ch_Jiasheng_EPFL_03_SideWork_08_TA_AlitumTemplate_DAB_Template_DAB_PCB.PcbLib:1739512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, symbol DAB_EE365:root_0_173951275_DAB_EE365.SchLib
- added R12, R2, R3, R4, R5, R6, R7, Rdiv1, Rdiv2, Rdiv3, Rdiv4, Rdiv5, Rdiv6, Rdiv7, Rdiv8, Rdiv9, Rfil1, Rfil2, Rfil3, Rfil4, Rfil5, Rfil6, Rfil8, Rfil9, Rsens1, Rsens2, Rsens3, Rsens4: Put Value here!, SM/1206, symbol DAB_EE365:root_2_Resistor (SMD)_DAB_EE365.SchLib
- added S1: TL3305BF100QG, C__Users_Jiasheng_OneDrive - epfl.ch_Documents_AltiumLL_SamacSys.PcbLib:TL3305BF160QG, symbol DAB_EE365:root_0_TL3305BF100QG_DAB_EE365.SchLib
- added Z1: 1N4750A-TR, C__Users_Jiasheng_OneDrive - epfl.ch_Documents_AltiumLL_SamacSys.PcbLib:DIOAD1310W86L370D235, symbol DAB_EE365:root_0_1N4750A-TR_DAB_EE365.SchLib
- gave numbers to parts that had none: 35
Connections:
- net ADCA0: now also C25.2, Rfil3.1
- net ADCA1: now also C20.2, R12.2
- net GND: now also C10.1, C11.1, C12.1, C13.1, C14.1, C15.1, C16.1, C17.1, C18.1, C19.1, C20.1, C25.1, C5.1, C6.1, C7.1, C8.1, C9.1, C_vdd5.1, C_vdd6.1, C_vdd8.1, C_vdd9.1, Csens1.1, Csens2.1, IC11.3 (INPUT), IC5.4 (GND), IC6.4 (GND), IC7.4 (GND), IC8.4 (GND), PS1.2 (GND), PS3.2 (GND), R5.1, R6.1, R7.1, Rdiv2.1, Rdiv4.1, Rdiv9.1, Z1.2 (A)
- net ac+: now also Rfil8.2
- net ac-: now also Rfil9.2
- net aux: now also IC12.8 (INPUT), Z1.1 (K)
- net prim+: now also C12.2, C13.2, PS1.1 (VIN), Rfil1.2, Rsens1.2
- net prim-: now also Rfil2.2
- net sec+: now also C4.1 (+), SWH?5.2 (D), SWH?7.2 (D), Shunt3.1, Rfil5.2; no longer J2.1, Shunt3.2
- net sec-: now also J2.1, Shunt3.2, Rfil6.2, Rsens3.2; no longer C4.1 (+), SWH?5.2 (D), SWH?7.2 (D), Shunt3.1
- net 12V renamed 12Vpri
- net 12Vpri: now also C10.2, C11.2, LED2.2 (A), PS1.3 (VOUT); no longer C_vdd3.2, C_vdd4.2, IC3.1 (VDD), IC4.1 (VDD), Rboot3.2, Rboot4.2
- new net: C_fil2.2, IC6.8 (V_IN+), Rfil5.1
- new net: IC8.3 (CMP_IN), Rdiv3.1, Rdiv4.2
- new net: LED1.1 (K), R5.2
- new net: D2.2 (A), IC7.6 (CMP_OUT), LED3.1 (K), Rdiv5.1
- new net: LED3.2 (A), Rdiv6.1
- new net: C_fil1.2, IC5.8 (V_IN+), Rfil1.1
- new net: IC9.6 (VOUT), R12.1, R2.2
- new net: D2.1 (K), D3.1 (K), Rdiv9.2
- new net: IC6.2 (OUT), Rfil4.2
- new net: C_fil2.1, IC6.7 (V_IN-), Rfil6.1
- new net: Csens1.2, D4.2 (A), IC9.3 (VIN+), Rsens1.1, Rsens2.2
- new net: C_fil1.1, IC5.7 (V_IN-), Rfil2.1
- new net: LED2.1 (K), R6.2
- new net: IC8.2 (OUT), Rdiv3.2
- new net: C_fil3.2, IC7.8 (V_IN+), IC8.7 (V_IN-), Rfil8.1
- new net: IC10.2 (VIN-), R3.1
- new net: Csens2.2, D5.2 (A), IC10.3 (VIN+), Rsens3.1, Rsens4.2
- new net: IC10.4 (VSS), Rsens4.1
- new net: IC10.6 (VOUT), R3.2, R4.1
- new net: IC9.2 (VIN-), R2.1
- new net: IC5.2 (OUT), Rfil3.2
- new net: IC7.5 (~{RESET}), IC8.5 (~{RESET}), S1.3, S1.4
- new net: C18.2, IC12.2 (COMMON_1), IC12.3 (COMMON_2)
- new net: C_fil3.1, IC7.7 (V_IN-), IC8.8 (V_IN+), Rfil9.1
- new net: C9.2, IC11.1 (ADJ/GND)
- new net: D3.2 (A), IC8.6 (CMP_OUT), LED4.1 (K), Rdiv7.1
- new net: LED4.2 (A), Rdiv8.1
- new net: IC7.3 (CMP_IN), Rdiv1.1, Rdiv2.2
- new net: IC7.2 (OUT), Rdiv1.2
- new net: IC9.4 (VSS), Rsens2.1
- new net: LED5.1 (K), R7.2
- new net: C19.2, IC12.6 (COMMON_3), IC12.7 (COMMON_4)
- new net 12Vsec: C16.2, C17.2, C_vdd3.2, C_vdd4.2, IC12.1 (OUTPUT), IC3.1 (VDD), IC4.1 (VDD), LED5.2 (A), PS3.3 (VOUT), Rboot3.2, Rboot4.2
- new net 3V3: C_vdd8.2, C_vdd9.2, IC10.7 (VDD), IC7.1 (V_S), IC8.1 (V_S), IC9.7 (VDD), Rdiv5.2, Rdiv6.2, Rdiv7.2, Rdiv8.2, S1.1, S1.2
- new net 3V3pri: C7.2, C8.2, C_vdd5.2, D4.1 (K), IC11.2 (OUTPUT), IC11.4 (VOUT), IC5.1 (V_S), LED1.2 (A)
- new net 3V3sec: C14.2, C15.2, C_vdd6.2, D5.1 (K), IC6.1 (V_S), PS3.1 (VIN)
- new net ADCB0: C5.2, Rfil4.1
- new net ADCB1: C6.2, R4.2
- no-connect marks 14 -> 28
Other:
- note added: "C_vdd???"
- note added: "Connect to..??"
- note added: "Correct RST???"
- note added: "Diode on which side ???"
- note added: "Heat sink???"
- note added: "TODO: add test points!"
- note added: "TODO: variable resistors ???!"

Commit message: correct input and output capcitors values from rapport1
Parts:
- renumbered J?1 to J1
Connections:
- net 3V3: no longer IC7.1 (V_S), IC8.1 (V_S), Rdiv5.2, Rdiv6.2, Rdiv7.2, Rdiv8.2, S1.1, S1.2
- net 3V3pri: now also IC7.1 (V_S), IC8.1 (V_S), Rdiv5.2, Rdiv6.2, Rdiv7.2, Rdiv8.2, S1.1, S1.2

Commit message: lined almost every footprint
Parts:
- removed C14, C15, C16, C24, C6, C7, C8, C_boot2, C_boot4, C_fil2, C_vdd4, C_vdd9, Chi5: Put Value Here!, C__Users_Jiasheng_OneDrive - epfl.ch_Jiasheng_EPFL_03_SideWork_08_TA_AlitumTemplate_DAB_Template_DAB_PCB.PcbLib:SM/1206, symbol DAB_EE365:root_1_Capacitor (SMD)_DAB_EE365.SchLib
- removed C23, C3: Put Value Here!, C__Users_Jiasheng_OneDrive - epfl.ch_Documents_AltiumLL_SamacSys.PcbLib:CAPPRD750W80D1625H3750, symbol DAB_EE365:root_3_UHW2A681MHD_DAB_EE365.SchLib
- removed D6: LMB14S-TP, C__Users_Jiasheng_OneDrive - epfl.ch_Documents_AltiumLL_SamacSys.PcbLib:LMB14STP, symbol DAB_EE365:root_0_LMB14S-TP_DAB_EE365.SchLib
- removed D7: ES2C, C__Users_Jiasheng_OneDrive - epfl.ch_Jiasheng_EPFL_03_SideWork_08_TA_Altium_Template_for_EE365_student_PCB1.PcbLib:DIOM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, symbol DAB_EE365:root_0_Schottky Diode_DAB_EE365.SchLib
- removed HS1: Heatsink, DAB_PCB:Heatsink FA-T220, symbol DAB_EE365:root_0_Heatsink_DAB_EE365.SchLib
- removed IC10, IC16: MCP6241-E_P, C__Users_Jiasheng_OneDrive - epfl.ch_Documents_AltiumLL_SamacSys.PcbLib:DIP781W56P254L950H533Q8N, symbol DAB_EE365:root_0_MCP6241-E_P_DAB_EE365.SchLib
- removed IC13: UCC27288DR, C__Users_Jiasheng_OneDrive - epfl.ch_Jiasheng_EPFL_03_SideWork_08_TA_Altium_Template_for_EE365_student_PCB1.PcbLib:SOIC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, symbol DAB_EE365:root_0_UCC27288DR_DAB_EE365.SchLib
- removed IC14: UA78L12ACDR, C__Users_Jiasheng_OneDrive - epfl.ch_Jiasheng_EPFL_03_SideWork_08_TA_Altium_Template_for_EE365_student_PCB1.PcbLib:SOIC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, symbol DAB_EE365:root_0_UA78L12ACDR_DAB_EE365.SchLib
- removed IC15: INA201AID, C__Users_Jiasheng_OneDrive - epfl.ch_Documents_AltiumLL_SamacSys.PcbLib:SOIC127P600X175-8N, symbol DAB_EE365:root_0_INA201AID_DAB_EE365.SchLib
- removed IC17: AZ1117IH-3.3TRG1, C__Users_Jiasheng_OneDrive - epfl.ch_Documents_AltiumLL_SamacSys.PcbLib:SOT230P700X180-4N, symbol DAB_EE365:root_0_AZ1117IH-3.3TRG1_DAB_EE365.SchLib
- removed L2: Inductor, symbol DAB_EE365:root_0_Inductor_DAB_EE365.SchLib
- removed LED4, LED5: WP710A10LGD, C__Users_Jiasheng_OneDrive - epfl.ch_Documents_AltiumLL_SamacSys.PcbLib:WP710A10LGD, symbol DAB_EE365:root_2_WP710A10LGD_DAB_EE365.SchLib
- removed PS2, PS3: 173951275, C__Users_Jiasheng_OneDrive - epfl.ch_Jiasheng_EPFL_03_SideWork_08_TA_AlitumTemplate_DAB_Template_DAB_PCB.PcbLib:1739512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, symbol DAB_EE365:root_0_173951275_DAB_EE365.SchLib
- removed R10, R9: Put Value here!, SM/1206, symbol DAB_EE365:root_3_Resistor (SMD)_DAB_EE365.SchLib
- removed R3, R4, R7, Rdiv7, Rdiv8, Rfil2, Rg5, Rgs5, Rhi5, Rsens3: Put Value here!, SM/1206, symbol DAB_EE365:root_2_Resistor (SMD)_DAB_EE365.SchLib
- removed S2: TL3305BF100QG, C__Users_Jiasheng_OneDrive - epfl.ch_Documents_AltiumLL_SamacSys.PcbLib:TL3305BF160QG, symbol DAB_EE365:root_0_TL3305BF100QG_DAB_EE365.SchLib
- removed SWH?9: MOSFET, C__Users_Jiasheng_OneDrive - epfl.ch_Jiasheng_EPFL_03_SideWork_08_TA_Altium_Template_for_EE365_student_PCB1.PcbLib:TO-2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, symbol DAB_EE365:root_0_NMOS-2_DAB_EE365.SchLib
- removed Shunt4: Put Value Here!, C__Users_Jiasheng_OneDrive - epfl.ch_Jiasheng_EPFL_03_SideWork_08_TA_AlitumTemplate_DAB_Template_DAB_PCB.PcbLib:CSNL251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, symbol DAB_EE365:root_0_ShuntResistor_DAB_EE365.SchLib
- removed Tr2: Transformer, C__Users_Jiasheng_OneDrive - epfl.ch_Jiasheng_EPFL_03_SideWork_08_TA_AlitumTemplate_DAB_Template_DAB_PCB.PcbLib:ETD39, symbol DAB_EE365:root_0_Transformer_DAB_EE365.SchLib
- removed Z2: 1N4750A-TR, C__Users_Jiasheng_OneDrive - epfl.ch_Documents_AltiumLL_SamacSys.PcbLib:DIOAD1310W86L370D235, symbol DAB_EE365:root_0_1N4750A-TR_DAB_EE365.SchLib
- added 4.7µF1, 4.7µF2, C10, C9: 10µF, Capacitor_SMD:C_1206_3216Metric, symbol DAB_EE365:root_1_Capacitor (SMD)_DAB_EE365.SchLib
- added C19: 1000pF, Capacitor_SMD:C_1206_3216Metric, symbol DAB_EE365:root_1_Capacitor (SMD)_DAB_EE365.SchLib
- added C_aux1: 22nF, Capacitor_SMD:C_2220_5750Metric, symbol DAB_EE365:root_1_Capacitor (SMD)_DAB_EE365.SchLib
- added C_boot1: 100nF, Capacitor_SMD:C_1206_3216Metric, symbol DAB_EE365:root_1_Capacitor (SMD)_DAB_EE365.SchLib
- added C_boot3: 0.22µF, Capacitor_SMD:C_1206_3216Metric, symbol DAB_EE365:root_1_Capacitor (SMD)_DAB_EE365.SchLib
- added C_fil3: 2.2µF, Capacitor_SMD:C_1206_3216Metric, symbol DAB_EE365:root_1_Capacitor (SMD)_DAB_EE365.SchLib
- added C_vdd3: 4.7µF, Capacitor_SMD:C_1206_3216Metric, symbol DAB_EE365:root_1_Capacitor (SMD)_DAB_EE365.SchLib
- added C_vdd8: Put Value Here!, Capacitor_SMD:C_1206_3216Metric, symbol DAB_EE365:root_1_Capacitor (SMD)_DAB_EE365.SchLib
- added Chi2: 22pF, Capacitor_SMD:C_1206_3216Metric, symbol DAB_EE365:root_1_Capacitor (SMD)_DAB_EE365.SchLib
- added HS1, HS2, HS3, HS4: Heatsink, DAB:Heatsink EA-T220, symbol DAB_EE365:Heatsink
- added IC13: MCP6241-E_P, DAB:DIP781W56P254L950H533Q8N, symbol DAB_EE365:root_0_MCP6241-E_P_DAB_EE365.SchLib
- added IC8: AZ1117IH-3.3TRG1, DAB:SOT230P700X180-4N, symbol DAB_EE365:root_0_AZ1117IH-3.3TRG1_DAB_EE365.SchLib
- added LED2, LED8, LED9: WP710A10LGD, DAB:WP710A10LID, symbol DAB_EE365:root_2_WP710A10LGD_DAB_EE365.SchLib
- added R10, R13: 680, Resistor_SMD:R_1206_3216Metric, symbol DAB_EE365:root_2_Resistor (SMD)_DAB_EE365.SchLib
- added R14, R18, Rgs1: 10k, Resistor_SMD:R_1206_3216Metric, symbol DAB_EE365:root_2_Resistor (SMD)_DAB_EE365.SchLib
- added R16, R20: 50, Resistor_SMD:R_1206_3216Metric, symbol DAB_EE365:root_2_Resistor (SMD)_DAB_EE365.SchLib
- added R6: 4.99k, Resistor_SMD:R_1206_3216Metric, symbol DAB_EE365:root_2_Resistor (SMD)_DAB_EE365.SchLib
- added R7, R8: 680, Resistor_SMD:R_1206_3216Metric, symbol DAB_EE365:root_3_Resistor (SMD)_DAB_EE365.SchLib
- added Rg1: 10, Resistor_SMD:R_1206_3216Metric, symbol DAB_EE365:root_2_Resistor (SMD)_DAB_EE365.SchLib
- added Rhi2: 2.2k, Resistor_SMD:R_1206_3216Metric, symbol DAB_EE365:root_2_Resistor (SMD)_DAB_EE365.SchLib
- added RrtE2: 10k, DAB:TRIMMER CT-6EP, symbol DAB_EE365:root_3_Variable Resistor_DAB_EE365.SchLib
- added Rsens2: 39.2k, Resistor_SMD:R_1206_3216Metric, symbol DAB_EE365:root_2_Resistor (SMD)_DAB_EE365.SchLib
- C11, C12, C13: value Put Value Here! -> 10µF; footprint C__Users_Jiasheng_OneDrive - epfl.ch_Jiasheng_EPFL_03_SideWork_08_TA_AlitumTemplate_DAB_Template_DAB_PCB.PcbLib:SM/1206 -> Capacitor_SMD:C_1206_3216Metric
- C14: renamed from C21; footprint C__Users_Jiasheng_OneDrive - epfl.ch_Jiasheng_EPFL_03_SideWork_08_TA_AlitumTemplate_DAB_Template_DAB_PCB.PcbLib:SM/1206 -> Resistor_SMD:R_1206_3216Metric
- C15: renamed from C22; footprint C__Users_Jiasheng_OneDrive - epfl.ch_Jiasheng_EPFL_03_SideWork_08_TA_AlitumTemplate_DAB_Template_DAB_PCB.PcbLib:SM/1206 -> Resistor_SMD:R_1206_3216Metric
- C16: renamed from C25; value Put Value Here! -> 1000pF; footprint C__Users_Jiasheng_OneDrive - epfl.ch_Jiasheng_EPFL_03_SideWork_08_TA_AlitumTemplate_DAB_Template_DAB_PCB.PcbLib:SM/1206 -> Capacitor_SMD:C_1206_3216Metric
- C17: value Put Value Here! -> 1000pF; footprint C__Users_Jiasheng_OneDrive - epfl.ch_Jiasheng_EPFL_03_SideWork_08_TA_AlitumTemplate_DAB_Template_DAB_PCB.PcbLib:SM/1206 -> Capacitor_SMD:C_1206_3216Metric
- C18: renamed from C20; value Put Value Here! -> 1000pF; footprint C__Users_Jiasheng_OneDrive - epfl.ch_Jiasheng_EPFL_03_SideWork_08_TA_AlitumTemplate_DAB_Template_DAB_PCB.PcbLib:SM/1206 -> Capacitor_SMD:C_1206_3216Metric
- C3: renamed from C2; footprint C__Users_Jiasheng_OneDrive - epfl.ch_Jiasheng_EPFL_03_SideWork_08_TA_AlitumTemplate_DAB_Template_DAB_PCB.PcbLib:SM/1206 -> Resistor_SMD:R_1206_3216Metric
- C4: renamed from C10; value Put Value Here! -> 10µF; footprint C__Users_Jiasheng_OneDrive - epfl.ch_Jiasheng_EPFL_03_SideWork_08_TA_AlitumTemplate_DAB_Template_DAB_PCB.PcbLib:SM/1206 -> Capacitor_SMD:C_1206_3216Metric
- C5: value Put Value Here! -> 0.1µF; footprint C__Users_Jiasheng_OneDrive - epfl.ch_Jiasheng_EPFL_03_SideWork_08_TA_AlitumTemplate_DAB_Template_DAB_PCB.PcbLib:SM/1206 -> Capacitor_SMD:C_1206_3216Metric
- C6: renamed from C18; value Put Value Here! -> 100nF; footprint C__Users_Jiasheng_OneDrive - epfl.ch_Jiasheng_EPFL_03_SideWork_08_TA_AlitumTemplate_DAB_Template_DAB_PCB.PcbLib:SM/1206 -> Capacitor_SMD:C_1206_3216Metric
- C7: renamed from C19; value Put Value Here! -> 330nF; footprint C__Users_Jiasheng_OneDrive - epfl.ch_Jiasheng_EPFL_03_SideWork_08_TA_AlitumTemplate_DAB_Template_DAB_PCB.PcbLib:SM/1206 -> Capacitor_SMD:C_1206_3216Metric
- C8: renamed from C9; value Put Value Here! -> 10µF; footprint C__Users_Jiasheng_OneDrive - epfl.ch_Jiasheng_EPFL_03_SideWork_08_TA_AlitumTemplate_DAB_Template_DAB_PCB.PcbLib:SM/1206 -> Capacitor_SMD:C_1206_3216Metric
- C_boot2: renamed from C_boot1; value Put Value Here! -> 100nF; footprint C__Users_Jiasheng_OneDrive - epfl.ch_Jiasheng_EPFL_03_SideWork_08_TA_AlitumTemplate_DAB_Template_DAB_PCB.PcbLib:SM/1206 -> Capacitor_SMD:C_1206_3216Metric; PART NUMBER (none) -> C1206C224K5RACTU
- C_boot4: renamed from C_boot3; value Put Value Here! -> 0.22µF; footprint C__Users_Jiasheng_OneDrive - epfl.ch_Jiasheng_EPFL_03_SideWork_08_TA_AlitumTemplate_DAB_Template_DAB_PCB.PcbLib:SM/1206 -> Capacitor_SMD:C_1206_3216Metric
- C_fil1: renamed from C_fil3; value Put Value Here! -> 2.2µF; footprint C__Users_Jiasheng_OneDrive - epfl.ch_Jiasheng_EPFL_03_SideWork_08_TA_AlitumTemplate_DAB_Template_DAB_PCB.PcbLib:SM/1206 -> Capacitor_SMD:C_1206_3216Metric
- C_fil2: renamed from C_fil1; value Put Value Here! -> 2.2µF; footprint C__Users_Jiasheng_OneDrive - epfl.ch_Jiasheng_EPFL_03_SideWork_08_TA_AlitumTemplate_DAB_Template_DAB_PCB.PcbLib:SM/1206 -> Capacitor_SMD:C_1206_3216Metric
- C_vdd1, C_vdd2: value Put Value Here! -> 2.2µF; footprint C__Users_Jiasheng_OneDrive - epfl.ch_Jiasheng_EPFL_03_SideWork_08_TA_AlitumTemplate_DAB_Template_DAB_PCB.PcbLib:SM/1206 -> Capacitor_SMD:C_1206_3216Metric; PART NUMBER (none) -> C1206C475K3PACTU
- C_vdd4: renamed from C_vdd3; value Put Value Here! -> 4.7µF; footprint C__Users_Jiasheng_OneDrive - epfl.ch_Jiasheng_EPFL_03_SideWork_08_TA_AlitumTemplate_DAB_Template_DAB_PCB.PcbLib:SM/1206 -> Capacitor_SMD:C_1206_3216Metric
- C_vdd5, C_vdd6: value Put Value Here! -> 10nF; footprint C__Users_Jiasheng_OneDrive - epfl.ch_Jiasheng_EPFL_03_SideWork_08_TA_AlitumTemplate_DAB_Template_DAB_PCB.PcbLib:SM/1206 -> Capacitor_SMD:C_1206_3216Metric
- C_vdd7: renamed from C_vdd8; footprint C__Users_Jiasheng_OneDrive - epfl.ch_Jiasheng_EPFL_03_SideWork_08_TA_AlitumTemplate_DAB_Template_DAB_PCB.PcbLib:SM/1206 -> Capacitor_SMD:C_1206_3216Metric
- Chi1: renamed from Chi2; value Put Value Here! -> 22pF; footprint C__Users_Jiasheng_OneDrive - epfl.ch_Jiasheng_EPFL_03_SideWork_08_TA_AlitumTemplate_DAB_Template_DAB_PCB.PcbLib:SM/1206 -> Capacitor_SMD:C_1206_3216Metric
- Chi3, Chi4, Cli1, Cli2, Cli3, Cli4: value Put Value Here! -> 22pF; footprint C__Users_Jiasheng_OneDrive - epfl.ch_Jiasheng_EPFL_03_SideWork_08_TA_AlitumTemplate_DAB_Template_DAB_PCB.PcbLib:SM/1206 -> Capacitor_SMD:C_1206_3216Metric
- Csens1: value Put Value Here! -> 4.7nF; footprint C__Users_Jiasheng_OneDrive - epfl.ch_Jiasheng_EPFL_03_SideWork_08_TA_AlitumTemplate_DAB_Template_DAB_PCB.PcbLib:SM/1206 -> Capacitor_SMD:C_1206_3216Metric
- Csens2: value Put Value Here! -> 2.2nF; footprint C__Users_Jiasheng_OneDrive - epfl.ch_Jiasheng_EPFL_03_SideWork_08_TA_AlitumTemplate_DAB_Template_DAB_PCB.PcbLib:SM/1206 -> Capacitor_SMD:C_1206_3216Metric
- D1: footprint C__Users_Jiasheng_OneDrive - epfl.ch_Documents_AltiumLL_SamacSys.PcbLib:LMB14STP -> DAB:LMB14STP
- D2, D3, D4, D5, Dboot1, Dboot2: footprint C__Users_Jiasheng_OneDrive - epfl.ch_Jiasheng_EPFL_03_SideWork_08_TA_Altium_Template_for_EE365_student_PCB1.PcbLib:DIOM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 -> DAB:DIOM5436X244N
- Dboot3: renamed from Dboot4; footprint C__Users_Jiasheng_OneDrive - epfl.ch_Jiasheng_EPFL_03_SideWork_08_TA_Altium_Template_for_EE365_student_PCB1.PcbLib:DIOM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 -> DAB:DIOM5436X244N
- Dboot4: renamed from Dboot3; footprint C__Users_Jiasheng_OneDrive - epfl.ch_Jiasheng_EPFL_03_SideWork_08_TA_Altium_Template_for_EE365_student_PCB1.PcbLib:DIOM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 -> DAB:DIOM5436X244N
- IC1, IC2: footprint C__Users_Jiasheng_OneDrive - epfl.ch_Jiasheng_EPFL_03_SideWork_08_TA_Altium_Template_for_EE365_student_PCB1.PcbLib:SOIC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 -> DAB:SOIC127P600X175-8N
- IC10: renamed from IC5; footprint C__Users_Jiasheng_OneDrive - epfl.ch_Documents_AltiumLL_SamacSys.PcbLib:SOIC127P600X175-8N -> DAB:SOIC127P600X175-8N
- IC11: renamed from IC6; footprint C__Users_Jiasheng_OneDrive - epfl.ch_Documents_AltiumLL_SamacSys.PcbLib:SOIC127P600X175-8N -> DAB:SOIC127P600X175-8N
- IC12: renamed from IC9; footprint C__Users_Jiasheng_OneDrive - epfl.ch_Documents_AltiumLL_SamacSys.PcbLib:DIP781W56P254L950H533Q8N -> DAB:DIP781W56P254L950H533Q8N
- IC3: renamed from IC4; footprint C__Users_Jiasheng_OneDrive - epfl.ch_Jiasheng_EPFL_03_SideWork_08_TA_Altium_Template_for_EE365_student_PCB1.PcbLib:SOIC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 -> DAB:SOIC127P600X175-8N
- IC4: renamed from IC3; footprint C__Users_Jiasheng_OneDrive - epfl.ch_Jiasheng_EPFL_03_SideWork_08_TA_Altium_Template_for_EE365_student_PCB1.PcbLib:SOIC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 -> DAB:SOIC127P600X175-8N
- IC5: renamed from IC12; footprint C__Users_Jiasheng_OneDrive - epfl.ch_Jiasheng_EPFL_03_SideWork_08_TA_Altium_Template_for_EE365_student_PCB1.PcbLib:SOIC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 -> DAB:SOIC127P600X175-8N
- IC6: renamed from IC7; footprint C__Users_Jiasheng_OneDrive - epfl.ch_Documents_AltiumLL_SamacSys.PcbLib:SOIC127P600X175-8N -> DAB:SOIC127P600X175-8N
- IC7: renamed from IC11; footprint C__Users_Jiasheng_OneDrive - epfl.ch_Documents_AltiumLL_SamacSys.PcbLib:SOT230P700X180-4N -> DAB:SOT230P700X180-4N
- IC9: renamed from IC8; footprint C__Users_Jiasheng_OneDrive - epfl.ch_Documents_AltiumLL_SamacSys.PcbLib:SOIC127P600X175-8N -> DAB:SOIC127P600X175-8N
- J1, J2: footprint C__Users_Jiasheng_OneDrive - epfl.ch_Jiasheng_EPFL_03_SideWork_08_TA_Altium_Template_for_EE365_student_PCB1.PcbLib:PHOE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 -> DAB:PHOENIX 1755736
- J3: renamed from J1; footprint DAB_EE365.PcbLib:3M_N3431-6302RB -> DAB:3M_N3431-6302RB
- LED1: renamed from LED6; footprint C__Users_Jiasheng_OneDrive - epfl.ch_Documents_AltiumLL_SamacSys.PcbLib:WP710A10LID -> DAB:WP710A10LID
- LED3: renamed from LED2; footprint C__Users_Jiasheng_OneDrive - epfl.ch_Documents_AltiumLL_SamacSys.PcbLib:WP710A10LGD -> DAB:WP710A10LID
- LED4: renamed from LED7; footprint C__Users_Jiasheng_OneDrive - epfl.ch_Documents_AltiumLL_SamacSys.PcbLib:WP710A10LGD -> DAB:WP710A10LID
- LED5: renamed from LED3; footprint C__Users_Jiasheng_OneDrive - epfl.ch_Documents_AltiumLL_SamacSys.PcbLib:WP710A10LGD -> DAB:WP710A10LID
- LED6: renamed from LED8; footprint C__Users_Jiasheng_OneDrive - epfl.ch_Documents_AltiumLL_SamacSys.PcbLib:WP710A10LGD -> DAB:WP710A10LID
- LED7: renamed from LED1; footprint C__Users_Jiasheng_OneDrive - epfl.ch_Documents_AltiumLL_SamacSys.PcbLib:WP710A10LGD -> DAB:WP710A10LID
- Me1, Me2, Me3, Me4: footprint M3 -> MountingHole:MountingHole_3.2mm_M3
- PS1: footprint C__Users_Jiasheng_OneDrive - epfl.ch_Jiasheng_EPFL_03_SideWork_08_TA_AlitumTemplate_DAB_Template_DAB_PCB.PcbLib:1739512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 -> DAB:173951275
- R1, Rboot1, Rboot2: footprint SM/1206 -> Resistor_SMD:R_1206_3216Metric
- R11, Rhi3, Rhi4, Rli1, Rli2, Rli3, Rli4: value Put Value here! -> 2.2k; footprint SM/1206 -> Resistor_SMD:R_1206_3216Metric
- R12: renamed from Rdiv9; value Put Value here! -> 200k; footprint SM/1206 -> Resistor_SMD:R_1206_3216Metric
- R15: renamed from Rfil3; value Put Value here! -> 50; footprint SM/1206 -> Resistor_SMD:R_1206_3216Metric
- R17: renamed from R2; value Put Value here! -> 10k; footprint SM/1206 -> Resistor_SMD:R_1206_3216Metric
- R19: renamed from R12; value Put Value here! -> 50; footprint SM/1206 -> Resistor_SMD:R_1206_3216Metric
- R2: renamed from R8; value Put Value here! -> 680; footprint SM/1206 -> Resistor_SMD:R_1206_3216Metric
- R3: renamed from Rdiv6; value Put Value here! -> 680; footprint SM/1206 -> Resistor_SMD:R_1206_3216Metric
- R4: renamed from Rdiv5; value Put Value here! -> 2.2k; footprint SM/1206 -> Resistor_SMD:R_1206_3216Metric
- R5: renamed from R6; value Put Value here! -> 4.99k; footprint SM/1206 -> Resistor_SMD:R_1206_3216Metric
- R9: renamed from R5; value Put Value here! -> 680; footprint SM/1206 -> Resistor_SMD:R_1206_3216Metric
- Rboot3: renamed from Rboot4; footprint SM/1206 -> Resistor_SMD:R_1206_3216Metric
- Rboot4: renamed from Rboot3; footprint SM/1206 -> Resistor_SMD:R_1206_3216Metric
- Rdiv1, Rdiv3: value Put Value here! -> 23.2k; footprint SM/1206 -> Resistor_SMD:R_1206_3216Metric
- Rdiv2, Rdiv4, Rgs2, Rgs3, Rgs4, Rgs6, Rgs7, Rgs8, Rsens4: value Put Value here! -> 10k; footprint SM/1206 -> Resistor_SMD:R_1206_3216Metric
- Rfil1: renamed from Rfil8; value Put Value here! -> 10; footprint SM/1206 -> Resistor_SMD:R_1206_3216Metric
- Rfil2: renamed from Rfil9; value Put Value here! -> 10; footprint SM/1206 -> Resistor_SMD:R_1206_3216Metric
- Rfil3: renamed from Rfil1; value Put Value here! -> 10; footprint SM/1206 -> Resistor_SMD:R_1206_3216Metric
- Rfil4, Rfil5, Rfil6, Rg2, Rg3, Rg4, Rg6, Rg7, Rg8: value Put Value here! -> 10; footprint SM/1206 -> Resistor_SMD:R_1206_3216Metric
- Rg5: renamed from Rg1; value Put Value here! -> 10; footprint SM/1206 -> Resistor_SMD:R_1206_3216Metric
- Rgs5: renamed from Rgs1; value Put Value here! -> 10k; footprint SM/1206 -> Resistor_SMD:R_1206_3216Metric
- Rhi1: renamed from Rhi2; value Put Value here! -> 2.2k; footprint SM/1206 -> Resistor_SMD:R_1206_3216Metric
- RrtE1: value Variable Resistor -> 10k; footprint TRIMMER CT-6EP -> DAB:TRIMMER CT-6EP
- Rsens1: value Put Value here! -> 97.6k; footprint SM/1206 -> Resistor_SMD:R_1206_3216Metric
- Rsens3: renamed from Rsens2; value Put Value here! -> 4.32k; footprint SM/1206 -> Resistor_SMD:R_1206_3216Metric
- S1: footprint C__Users_Jiasheng_OneDrive - epfl.ch_Documents_AltiumLL_SamacSys.PcbLib:TL3305BF160QG -> DAB:TL3305BF160QG
- SWH?1, SWH?6, SWH?8: footprint C__Users_Jiasheng_OneDrive - epfl.ch_Jiasheng_EPFL_03_SideWork_08_TA_Altium_Template_for_EE365_student_PCB1.PcbLib:TO-2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 -> DAB:TO-220AB
- SWH?2: renamed from SWH?3; footprint C__Users_Jiasheng_OneDrive - epfl.ch_Jiasheng_EPFL_03_SideWork_08_TA_Altium_Template_for_EE365_student_PCB1.PcbLib:TO-2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 -> DAB:TO-220AB
- SWH?3: renamed from SWH?5; footprint C__Users_Jiasheng_OneDrive - epfl.ch_Jiasheng_EPFL_03_SideWork_08_TA_Altium_Template_for_EE365_student_PCB1.PcbLib:TO-2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 -> DAB:TO-220AB
- SWH?4: renamed from SWH?7; footprint C__Users_Jiasheng_OneDrive - epfl.ch_Jiasheng_EPFL_03_SideWork_08_TA_Altium_Template_for_EE365_student_PCB1.PcbLib:TO-2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 -> DAB:TO-220AB
- SWH?5: renamed from SWH?2; footprint C__Users_Jiasheng_OneDrive - epfl.ch_Jiasheng_EPFL_03_SideWork_08_TA_Altium_Template_for_EE365_student_PCB1.PcbLib:TO-2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 -> DAB:TO-220AB
- SWH?7: renamed from SWH?4; footprint C__Users_Jiasheng_OneDrive - epfl.ch_Jiasheng_EPFL_03_SideWork_08_TA_Altium_Template_for_EE365_student_PCB1.PcbLib:TO-2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 -> DAB:TO-220AB
- Shunt1: value Put Value Here! -> 25m; footprint C__Users_Jiasheng_OneDrive - epfl.ch_Jiasheng_EPFL_03_SideWork_08_TA_AlitumTemplate_DAB_Template_DAB_PCB.PcbLib:CSNL251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 -> Resistor_SMD:R_2512_6332Metric
- Shunt2: renamed from Shunt3; value Put Value Here! -> 10m; footprint C__Users_Jiasheng_OneDrive - epfl.ch_Jiasheng_EPFL_03_SideWork_08_TA_AlitumTemplate_DAB_Template_DAB_PCB.PcbLib:CSNL251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 -> Resistor_SMD:R_2512_6332Metric
- Shunt3: renamed from Shunt2; value Put Value Here! -> 10m; footprint C__Users_Jiasheng_OneDrive - epfl.ch_Jiasheng_EPFL_03_SideWork_08_TA_AlitumTemplate_DAB_Template_DAB_PCB.PcbLib:CSNL251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 -> Resistor_SMD:R_2512_6332Metric
- Tr1: footprint C__Users_Jiasheng_OneDrive - epfl.ch_Jiasheng_EPFL_03_SideWork_08_TA_AlitumTemplate_DAB_Template_DAB_PCB.PcbLib:ETD39 -> DAB:B66362X1014T001
- Z1: footprint C__Users_Jiasheng_OneDrive - epfl.ch_Documents_AltiumLL_SamacSys.PcbLib:DIOAD1310W86L370D235 -> DAB:DIOAD1310W86L370D235
- renumbered C4 to C2, J3 to TP1
Connections:
- net 3V3 is gone; now on net 3V3pri: C_vdd7.2, IC12.7 (VDD)
- net 12Vpri: now also C5.2, C6.2, C8.2, C_vdd4.2, IC3.1 (VDD), IC4.1 (VDD), IC5.1 (OUTPUT), IC7.1 (ADJ/GND), Rboot3.2, Rboot4.2, C_vdd3.2, IC8.1 (ADJ/GND), LED2.2 (A)
- net 3V3pri: now also IC6.5 (~{RESET}), IC9.5 (~{RESET}), R11.2, S1.3, S1.4, C10.2, C9.2, R10.2; no longer S1.1, S1.2
- net 3V3sec: now also C12.2, C13.2, C_vdd8.2, IC13.7 (VDD), IC8.2 (OUTPUT), IC8.4 (VOUT), LED8.2 (A)
- net ADCB0: now also C17.2, R16.1; no longer C5.2, Rfil4.1
- net ADCB1: now also C19.2, R20.2
- net CS1_ISO: now also R7.2
- net CS2_ISO: now also R8.2
- net GND: now also IC5.2 (COMMON_1), IC5.3 (COMMON_2), IC5.6 (COMMON_3), IC5.7 (COMMON_4), Rgs3.1, 4.7µF1.1, 4.7µF2.1, C10.1, C19.1, C9.1, C_aux1.1, C_vdd3.1, C_vdd8.1, Chi2.1, IC8.3 (INPUT), R13.1, R14.1, R6.1, Rgs1.1; no longer Rgs6.1, Rgs8.1
- net PWM2B_ISO: now also Rhi2.2; no longer Rhi3.2
- net PWM3A_ISO: now also Rli4.2; no longer Rli3.2
- net PWM4A_ISO: now also Rli3.2; no longer Rli4.2
- net PWM4B_ISO: now also Rhi3.2
- net ac+: now also Tr1.2; no longer Tr1.8
- net ac-: now also Rgs6.1, C_boot1.1; no longer Rgs3.1
- net aux: now also C7.2, C_aux1.2
- net prim+: now also 4.7µF1.2, 4.7µF2.2; no longer C12.2, C13.2
- net prim-: now also Rfil5.2
- net sec+: now also Rfil4.2; no longer Rfil5.2
- net sec-: now also Rsens2.2
- net vg2: now also Rg1.1, Rgs1.2; no longer Rg2.2, Rgs2.2
- net vg3: now also Rg6.2, Rgs6.2; no longer Rg3.2, Rgs3.2
- net vg4: now also Rg2.1, Rgs2.2; no longer Rg4.2, Rgs4.2
- net vg5: now also Rg8.2, Rgs8.2
- net vg6: now also Rg4.1, Rgs4.2; no longer Rg6.2, Rgs6.2
- net vg8: now also Rg3.1, Rgs3.2; no longer Rg8.2, Rgs8.2
- net vs5: now also Rgs8.1, Tr1.13 (1); no longer Tr1.16
- net vs7: now also Tr1.1, C_boot3.1; no longer Tr1.13
- net at IC11.8 (V_IN+): now also Rfil4.1, C_fil3.2; no longer Rfil5.1
- net at Cli4.2, Rli4.1: now also IC4.6 (LI); no longer IC3.6 (LI)
- net at IC11.2 (OUT): now also R16.2; no longer Rfil4.2
- net at IC11.7 (V_IN-), Rfil6.1: now also C_fil3.1
- net at IC4.3 (HO): now also Rg8.1
- net at C_fil2.1, IC10.7 (V_IN-): now also Rfil5.1
- net at D1.2 (AC_1): now also Tr1.14; no longer Tr1.11
- net at D1.3 (AC_2): now also Tr1.10; no longer Tr1.9
- net at IC9.2 (OUT): now also RrtE2.1; no longer Rdiv3.2
- net at Csens2.2, D5.2 (A), Rsens4.2: now also IC13.3 (VIN+), Rsens2.1
- net at Rsens4.1: now also IC13.4 (VSS)
- net at L1.2: now also Tr1.6; no longer Tr1.1
- net at Cli3.2, Rli3.1: now also IC3.6 (LI); no longer IC4.6 (LI)
- net at Dboot3.1 (K), IC3.2 (HB): now also C_boot3.2
- net at IC3.5 (HI): now also Chi3.2, Rhi3.1
- net at IC3.8 (LO): now also Rg3.2; no longer Rg8.1
- net at RrtE1.1: now also IC6.2 (OUT)
- net at RrtE1.2: now also Rdiv1.2
- net at IC1.8 (LO): now also Rg1.2; no longer Rg2.1
- net at Rg6.1: now also IC2.3 (HO); no longer IC4.8 (LO)
- net at R11.1: now also D3.2 (A), IC9.6 (CMP_OUT), LED9.1 (K)
- net at Dboot2.1 (K), IC2.2 (HB): now also C_boot1.2
- net at IC2.8 (LO): now also Rg2.2; no longer Rg4.1
- net at LED6.2 (A): now also R8.1
- net at LED4.2 (A): now also R7.1
- removed net 12Vsec: C17.2, C_vdd4.2, IC3.1 (VDD), IC4.1 (VDD), IC5.1 (OUTPUT), Rboot3.2, Rboot4.2
- new net: IC13.6 (VOUT), R18.2, R20.1
- new net: R14.2, S1.1, S1.2
- new net: Chi2.2, IC2.5 (HI), Rhi2.1
- new net: LED2.1 (K), R6.2
- new net: LED8.1 (K), R13.2
- new net: IC4.8 (LO), Rg4.2
- new net: LED9.2 (A), R10.1
- new net: Rdiv3.2, RrtE2.2
- new net: IC13.2 (VIN-), R18.1
Other:
- note added: "Conntector type?"
- note added: "TODO: 3d mosfet"
- note added: "TODO: boot res"
- note added: "TODO: induct footprint"
- note added: "TODO: inptut capcas"
- note added: "aux, prim+ also ^ ???"
- note added: "same filter???"
- note removed: "Components Library"
- note removed: "TODO: variable resistors ???!"
- moved on the sheet: C18, C_boot2, C_fil2, C_vdd5, LED1, LED4, R17, Rdiv1, Rg5, TP1, Tr1

Commit message: added testpoints
Parts:
- removed 4.7µF1: 10µF, Capacitor_SMD:C_1206_3216Metric, symbol DAB_EE365:root_1_Capacitor (SMD)_DAB_EE365.SchLib
- removed IC7, IC8: AZ1117IH-3.3TRG1, DAB:SOT230P700X180-4N, symbol DAB_EE365:root_0_AZ1117IH-3.3TRG1_DAB_EE365.SchLib
- added C20: 22µF, Capacitor_SMD:C_2220_5750Metric, symbol DAB_EE365:root_1_Capacitor (SMD)_DAB_EE365.SchLib
- added C21: 4.7µF, Capacitor_SMD:C_1206_3216Metric, symbol DAB_EE365:root_1_Capacitor (SMD)_DAB_EE365.SchLib
- added C_vdd10, C_vdd9: 10nF, Capacitor_SMD:C_1206_3216Metric, symbol DAB_EE365:root_1_Capacitor (SMD)_DAB_EE365.SchLib
- added IC14, IC15: (no value), DAB:SOT230P700X180-4N, symbol DAB_EE365:AZ1117IH-3.3TRG1
- added TP10: sec, Connector_PinHeader_2.54mm:PinHeader_1x02_P2.54mm_Vertical, symbol DAB_EE365:root_0_Test point_DAB_EE365.SchLib
- added TP11: ac, Connector_PinHeader_2.54mm:PinHeader_1x02_P2.54mm_Vertical, symbol DAB_EE365:root_0_Test point_DAB_EE365.SchLib
- added TP12, TP18: TP?, symbol Connector:Conn_01x03_Pin
- added TP13: Vaux, Connector_PinHeader_2.54mm:PinHeader_1x02_P2.54mm_Vertical, symbol DAB_EE365:root_0_Test point_DAB_EE365.SchLib
- added TP14: I_prim, Connector_PinHeader_2.54mm:PinHeader_1x02_P2.54mm_Vertical, symbol DAB_EE365:root_0_Test point_DAB_EE365.SchLib
- added TP15: I_ac, Connector_PinHeader_2.54mm:PinHeader_1x02_P2.54mm_Vertical, symbol DAB_EE365:root_0_Test point_DAB_EE365.SchLib
- added TP16: I_sec, Connector_PinHeader_2.54mm:PinHeader_1x02_P2.54mm_Vertical, symbol DAB_EE365:root_0_Test point_DAB_EE365.SchLib
- added TP17: Conn_01x10_Pin, Connector_PinHeader_2.54mm:PinHeader_1x10_P2.54mm_Vertical, symbol Connector:Conn_01x10_Pin
- added TP2: Vds3, Connector_PinHeader_2.54mm:PinHeader_1x02_P2.54mm_Vertical, symbol DAB_EE365:root_0_Test point_DAB_EE365.SchLib
- added TP3: Vds5, Connector_PinHeader_2.54mm:PinHeader_1x02_P2.54mm_Vertical, symbol DAB_EE365:root_0_Test point_DAB_EE365.SchLib
- added TP4: Vds7, Connector_PinHeader_2.54mm:PinHeader_1x02_P2.54mm_Vertical, symbol DAB_EE365:root_0_Test point_DAB_EE365.SchLib
- added TP5: Vgs2, Connector_PinHeader_2.54mm:PinHeader_1x02_P2.54mm_Vertical, symbol DAB_EE365:root_0_Test point_DAB_EE365.SchLib
- added TP6: Vgs4, Connector_PinHeader_2.54mm:PinHeader_1x02_P2.54mm_Vertical, symbol DAB_EE365:root_0_Test point_DAB_EE365.SchLib
- added TP7: Vgs6, Connector_PinHeader_2.54mm:PinHeader_1x02_P2.54mm_Vertical, symbol DAB_EE365:root_0_Test point_DAB_EE365.SchLib
- added TP8: Vgs8, Connector_PinHeader_2.54mm:PinHeader_1x02_P2.54mm_Vertical, symbol DAB_EE365:root_0_Test point_DAB_EE365.SchLib
- added TP9: prim, Connector_PinHeader_2.54mm:PinHeader_1x02_P2.54mm_Vertical, symbol DAB_EE365:root_0_Test point_DAB_EE365.SchLib
- C1: value Put Value Here! -> 680µF; footprint C__Users_Jiasheng_OneDrive - epfl.ch_Documents_AltiumLL_SamacSys.PcbLib:CAPPRD750W80D1625H3750 -> DAB:CAPPRD750W80D1625H3750
- C2: value Put Value Here! -> 1000µF; footprint C__Users_Jiasheng_OneDrive - epfl.ch_Documents_AltiumLL_SamacSys.PcbLib:CAPPRD750W80D1625H3750 -> DAB:MAL215097614E3; MANUFACTURER_NAME Nichicon -> Vishay; MANUFACTURER_PART_NUMBER UHW2A681MHD -> MAL215097614E3; MOUSER PART NUMBER 647-UHW2A681MHD -> 594-MAL215097614E3; MOUSER PRICE/STOCK https://www.mouser.co.uk/ProductDetail/Nichicon/UHW2A681MHD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 -> https://www.mouser.ch/ProductDetail/Vishay-BC-Components/MA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
- C22: renamed from 4.7µF2; value 10µF -> 4.7µF; PART NUMBER (none) -> GRM31CZ72A475KE1
- C3: value Put Value Here! -> 22µF; footprint Resistor_SMD:R_1206_3216Metric -> Capacitor_SMD:C_2220_5750Metric; PART NUMBER (none) -> C5750X7S2A226M280KB
- C_aux1: PART NUMBER (none) -> C5750X7S2A226M280KB
- C_vdd7, C_vdd8: value Put Value Here! -> 1µF
- HS1, HS2, HS3, HS4: footprint DAB:Heatsink EA-T220 -> DAB:FAT22025E
- J1, J2: value ${FAMILY} -> (none)
- R1: value Put Value here! -> 27.4k
- Rboot1, Rboot2: value Put Value here! -> 10
- Rboot3, Rboot4: value Put Value here! -> 4.99
- SWH1: renamed from SWH?1; value MOSFET -> PHP18NQ11T
- SWH2: renamed from SWH?2; value MOSFET -> PHP18NQ11T
- SWH3: renamed from SWH?3; value MOSFET -> IRLB8743PbF
- SWH4: renamed from SWH?4; value MOSFET -> IRLB8743PbF
- SWH5: renamed from SWH?5; value MOSFET -> PHP18NQ11T
- SWH6: renamed from SWH?6; value MOSFET -> IRLB8743PbF
- SWH7: renamed from SWH?7; value MOSFET -> PHP18NQ11T
- SWH8: renamed from SWH?8; value MOSFET -> IRLB8743PbF
- TP1: value Test point -> Vds1; footprint C__Users_Jiasheng_OneDrive - epfl.ch_Documents_AltiumLL_SamacSys.PcbLib:HDRV2W64P0X508_1X2_1016X254X838P -> Connector_PinHeader_2.54mm:PinHeader_1x02_P2.54mm_Vertical
Connections:
- net 12Vpri: now also IC14.3 (INPUT), IC15.3 (INPUT), TP12.1 (Pin_1), TP18.1 (Pin_1)
- net 3V3pri: now also C_vdd10.2, C_vdd9.2, IC14.2 (OUTPUT), IC14.4 (VOUT), TP18.2 (Pin_2)
- net 3V3sec: now also IC15.2 (OUTPUT), IC15.4 (VOUT), TP12.2 (Pin_2)
- net ADCA1: now also TP14.1
- net ADCB1: now also TP16.1
- net ECAP2_ISO: now also D2.1 (K), D3.1 (K), R12.2, TP15.1
- net GND: now also TP1.2, C20.1, C21.1, C_vdd10.1, C_vdd9.1, IC14.1 (ADJ/GND), IC15.1 (ADJ/GND), TP12.3 (Pin_3), TP13.2, TP14.2, TP15.2, TP16.2, TP17.1 (Pin_1), TP17.10 (Pin_10), TP18.3 (Pin_3), TP2.2, TP3.2, TP4.2, TP5.2, TP6.2, TP7.2, TP8.2
- net PWM1A_ISO: now also TP17.2 (Pin_2)
- net PWM1B_ISO: now also TP17.6 (Pin_6)
- net PWM2A_ISO: now also TP17.3 (Pin_3)
- net PWM2B_ISO: now also TP17.7 (Pin_7)
- net PWM3A_ISO: now also TP17.4 (Pin_4)
- net PWM3B_ISO: now also TP17.8 (Pin_8)
- net PWM4A_ISO: now also TP17.5 (Pin_5)
- net PWM4B_ISO: now also TP17.9 (Pin_9)
- net ac+: now also TP11.1
- net ac-: now also TP11.2, TP2.1
- net aux: now also TP13.1
- net prim+: now also C21.2, TP9.1
- net prim-: now also C20.2, TP9.2
- net sec+: now also TP10.1
- net sec-: now also TP10.2
- net vg2: now also TP5.1
- net vg4: now also TP6.1
- net vg6: now also TP7.1
- net vg8: now also TP8.1
- net vs1: now also TP1.1
- net vs5: now also TP3.1
- net vs7: now also TP4.1
- no-connect marks 28 -> 38
Other:
- note added: "same filter??? -> no!"
- note removed: "C_vdd???"
- note removed: "Connect to..??"
- note removed: "Conntector type?"
- note removed: "Correct RST???"
- note removed: "Different GND for Prim and Sec???"
- note removed: "Diode on which side ???"
- note removed: "Heat sink???"
- note removed: "TODO: 3d mosfet"
- note removed: "TODO: add test points!"
- note removed: "TODO: boot res"
- note removed: "TODO: inptut capcas"
- note removed: "aux, prim+ also ^ ???"
- note removed: "same filter???"
- moved on the sheet: C1, HS1, R1, RrtE1, TP1
